Commit message: Update ar_macro.xacro
updated joint limits again... left the moments of inertia alone, could be close enough, did not update joint 6 position, may have to move x up by 5 mm, to be seen.

File: ar_description/urdf/ar_macro.xacro (robot description, xacro)
@@ -143,5 +143,5 @@
       <child link="link_4"/>
       <axis xyz="0 0 -1"/>
-      <limit lower="${-165.0 / 180.0 * pi}" upper="${165.0 / 180.0 * pi}" effort="0" velocity="0.5"/>
+      <limit lower="${-180 / 180.0 * pi}" upper="${180 / 180.0 * pi}" effort="0" velocity="0.5"/>
     </joint>
     <link name="link_5">
@@ -201,5 +201,5 @@
       <child link="link_6"/>
       <axis xyz="0 0 1"/>
-      <limit lower="${-155.0 / 180.0 * pi}" upper="${155.0 / 180.0 * pi}" effort="0" velocity="1.0"/>
+      <limit lower="${-180 / 180.0 * pi}" upper="${180 / 180.0 * pi}" effort="0" velocity="1.0"/>
     </joint>
     <!-- center of the end effector mounting surface on link_6 -->

Commit message: Update ar_macro.xacro
updated joint 5 position

File: ar_description/urdf/ar_macro.xacro (robot description, xacro)
@@ -147,5 +147,5 @@
     <link name="link_5">
       <inertial>
-        <origin rpy="0 0 0" xyz="0.0015066 -1.3102E-05 -0.012585"/>
+        <origin rpy="0 0 0" xyz="0 0 -0.0275/>
         <mass value="0.11562"/>
         <inertia ixx="5.5035E-05" ixy="-1.019E-08" ixz="-2.6243E-06" iyy="8.2921E-05" iyz="1.4437E-08" izz="5.2518E-05"/>

Commit message: Update ar_macro.xacro

File: ar_description/urdf/ar_macro.xacro (robot description, xacro)
@@ -147,5 +147,5 @@
     <link name="link_5">
       <inertial>
-        <origin rpy="0 0 0" xyz="0 0 -0.0275/>
+        <origin rpy="0 0 0" xyz="0 0 -0.0275"/>
         <mass value="0.11562"/>
         <inertia ixx="5.5035E-05" ixy="-1.019E-08" ixz="-2.6243E-06" iyy="8.2921E-05" iyz="1.4437E-08" izz="5.2518E-05"/>

Commit message: Update ar_macro.xacro

File: ar_description/urdf/ar_macro.xacro (robot description, xacro)
@@ -168,5 +168,5 @@
     </link>
     <joint name="joint_5" type="revolute">
-      <origin rpy="${pi} 0 -1.5708" xyz="0 0 -0.22263"/>
+      <origin rpy="${pi} 0 -1.5708" xyz=""2.9287E-10 -1.6472E-09 0.0091432"/>
       <parent link="link_4"/>
       <child link="link_5"/>

Commit message: Update ar_macro.xacro

File: ar_description/urdf/ar_macro.xacro (robot description, xacro)
@@ -168,5 +168,5 @@
     </link>
     <joint name="joint_5" type="revolute">
-      <origin rpy="${pi} 0 -1.5708" xyz=""2.9287E-10 -1.6472E-09 0.0091432"/>
+      <origin rpy="${pi} 0 -1.5708" xyz="2.9287E-10 -1.6472E-09 0.0091432"/>
       <parent link="link_4"/>
       <child link="link_5"/>

Commit message: Update ar_macro.xacro

File: ar_description/urdf/ar_macro.xacro (robot description, xacro)
@@ -168,5 +168,5 @@
     </link>
     <joint name="joint_5" type="revolute">
-      <origin rpy="${pi} 0 -1.5708" xyz="2.9287E-10 -1.6472E-09 0.0091432"/>
+      <origin rpy="${pi} 0 -1.5708" xyz=""0 0 -0.22263"/>
       <parent link="link_4"/>
       <child link="link_5"/>

Commit message: Update ar_macro.xacro

File: ar_description/urdf/ar_macro.xacro (robot description, xacro)
@@ -147,5 +147,5 @@
     <link name="link_5">
       <inertial>
-        <origin rpy="0 0 0" xyz="0 0 -0.0275"/>
+        <origin rpy="0 0 0" xyz="0.0015066 -1.3102E-05 -0.012585"/>
         <mass value="0.11562"/>
         <inertia ixx="5.5035E-05" ixy="-1.019E-08" ixz="-2.6243E-06" iyy="8.2921E-05" iyz="1.4437E-08" izz="5.2518E-05"/>

Commit message: Update ar_macro.xacro

File: ar_description/urdf/ar_macro.xacro (robot description, xacro)
@@ -168,5 +168,5 @@
     </link>
     <joint name="joint_5" type="revolute">
-      <origin rpy="${pi} 0 -1.5708" xyz=""0 0 -0.22263"/>
+      <origin rpy="${pi} 0 -1.5708" xyz="0 0 -0.22263"/>
       <parent link="link_4"/>
       <child link="link_5"/>

Commit message: Update ar_macro.xacro

File: ar_description/urdf/ar_macro.xacro (robot description, xacro)
@@ -197,5 +197,5 @@
     </link>
     <joint name="joint_6" type="revolute">
-      <origin rpy="0 0 3.1416" xyz="0.000 0 0.03625"/>
+      <origin rpy="0 0 3.1416" xyz="0.000 0 0.042"/>
       <parent link="link_5"/>
       <child link="link_6"/>

Commit message: Update ar_macro.xacro

File: ar_description/urdf/ar_macro.xacro (robot description, xacro)
@@ -197,5 +197,5 @@
     </link>
     <joint name="joint_6" type="revolute">
-      <origin rpy="0 0 3.1416" xyz="0.000 0 0.042"/>
+      <origin rpy="0 0 3.1416" xyz="0.000 0 0.025"/>
       <parent link="link_5"/>
       <child link="link_6"/>

Commit message: finishing updating the offsets for joint 6.

File: ar_description/urdf/ar_macro.xacro (robot description, xacro)
@@ -208,5 +208,5 @@
       <parent link="link_6" />
       <child link="ee_link" />
-      <origin xyz="0 0 0.0" rpy="0 0 0" />
+      <origin xyz="0 0 0.0170" rpy="0 0 0" />
     </joint>
   </xacro:macro>
